File: _autosave-Osciliscope.kicad_sch (KiCad schematic)
At the start: 25 parts, among them J1 U.FL, J2 Conn_01x04_Socket, J3 U.FL, J4 Conn_01x04_Socket, SW1 SW_Rotary_1x8_MP, SW2 SW_Rotary_1x8_MP, U1 MCP1700x-330xxMB, U2 ADC082S101, U5 TLV9061xDBV, U7 TLV9061xDBV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

Commit message: Added new op amp design
Other:
- note added: "FUSB307B PD"
- note added: "FUSB307B PD + USB-C"
Changed lines of the file:
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@@
 	(generator_version "9.0")
 	(paper "A4")
+	(text "FUSB307B PD + USB-C"
+		(exclude_from_sim no)
+		(at 182 46.5 0)
+		(effects
+			(font
+				(size 1.27 1.27)
+			)
+		)
+	)
+	(text "FUSB307B PD"
+		(exclude_from_sim no)
+		(at 268.5 11.5 0)
+		(effects
+			(font
+				(size 1.27 1.27)
+			)
+		)
+	)
+	(text "FUSB307B PD + USB-C"
+		(exclude_from_sim no)
+		(at 268.5 11.5 0)
+		(effects
+			(font
+				(size 1.27 1.27)
+			)
+		)
+	)
 	(junction
 		(at 119.38 58.42)
@@
 		)
 	)
+	(polyline
+		(pts
+			(xy 287 50) (xy 250 50)
+		)
+		(stroke
+			(width 0)
+			(type default)
+		)
+	)
+	(polyline
+		(pts
+			(xy 287 50) (xy 250 50)
+		)
+		(stroke
+			(width 0)
+			(type default)
+		)
+	)
 	(wire
 		(pts
@@
 		)
 	)
+	(polyline
+		(pts
+			(xy 250 50) (xy 250 10)
+		)
+		(stroke
+			(width 0)
+			(type default)
+		)
+	)
+	(polyline
+		(pts
+			(xy 250 10) (xy 287 10)
+		)
+		(stroke
+			(width 0)
+			(type default)
+		)
+	)
 	(wire
 		(pts
@@
 		)
 	)
+	(polyline
+		(pts
+			(xy 250 50) (xy 250 10)
+		)
+		(stroke
+			(width 0)
+			(type default)
+		)
+	)
 	(wire
 		(pts
@@
 		)
 	)
+	(polyline
+		(pts
+			(xy 250 10) (xy 287 10)
+		)
+		(stroke
+			(width 0)
+			(type default)
+		)
+	)
+	(polyline
+		(pts
+			(xy 287 10) (xy 287 50)
+		)
+		(stroke
+			(width 0)
+			(type default)
+		)
+	)
+	(polyline
+		(pts
+			(xy 287 10) (xy 287 50)
+		)
+		(stroke
+			(width 0)
+			(type default)
+		)
+	)
 	(wire
 		(pts
@@
 		)
 	)
+	(polyline
+		(pts
+			(xy 132 45) (xy 232 45)
+		)
+		(stroke
+			(width 0)
+			(type default)
+		)
+	)
 	(wire
 		(pts
@@
 		)
 	)
+	(polyline
+		(pts
+			(xy 232 45) (xy 232 145)
+		)
+		(stroke
+			(width 0)
+			(type default)
+		)
+	)
 	(wire
 		(pts
@@
 		)
 		(stroke
+			(width 0)
+			(type default)
+		)
+	)
+	(polyline
+		(pts
+			(xy 232 145) (xy 132 145)
+		)
+		(stroke
+			(width 0)
+			(type default)
+		)
+	)
+	(polyline
+		(pts
+			(xy 132 145) (xy 132 45)
+		)
+		(stroke

Commit message: PCB design
Parts:
- removed C2: 1uF, Capacitor_SMD:C_1206_3216Metric, symbol Device:C
- added C10, C9: 1u, Capacitor_SMD:C_1206_3216Metric, symbol Device:C
- added D1, D2, D3, D4: D, Diode_SMD:D_0201_0603Metric, symbol Device:D
- added SW3, SW4: SW_Nidec_CAS-120A1, Button_Switch_SMD:Nidec_Copal_CAS-120A, symbol Switch:SW_Nidec_CAS-120A1
Connections:
- net 3.3Vo is gone; now on net V3.3: C3.1, U2.2 (V_{A})
- net GND: now also D2.2 (A), D4.2 (A)
- net V3.3: now also D1.1 (K), D3.1 (K)
- net at J1.1 (In), R10.1: now also C9.1, SW3.3 (A); no longer R3.2
- net at J3.1 (In), R14.1: now also C10.1, SW4.3 (A); no longer R4.2
- new net: D3.2 (A), D4.1 (K), R4.2, SW4.2 (B)
- new net: C10.2, SW4.1 (C)
- new net: D1.2 (A), D2.1 (K), R3.2, SW3.2 (B)
- new net: C9.2, SW3.1 (C)
Other:
- note removed: "FUSB307B PD"
- note removed: "FUSB307B PD + USB-C"
- moved on the sheet: J1, J3, R10, R14, R3, R4, U5, U7
