File: Osciliscope.kicad_pcb (KiCad board)
At the start: 2 copper layers, 51 x 102 mm, 67 parts, among them J1 Conn_01x09_Socket, J2 Conn_01x04_Socket, J3 U.FL, J5 USB_C_Receptacle_USB2.0_14P, J6 Conn_01x02_MountingPin, J7 U.FL, J8 USB_C_Receptacle_USB2.0_14P, J9 Conn_01x03_Socket, SW1 RotaryEncoder_Switch, SW4 SW_Nidec_CAS-120A1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

Commit message: Footprint updates
Connections:
- R3 pad 2: Net-(SW7-C) -> Net-(R3-Pad2)
- R4 pad 2: Net-(SW4-C) -> Net-(R4-Pad2)
Changed lines of the file:
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@@
 	(net 46 "Net-(SW7-C)")
 	(net 47 "V1.65RAW")
+	(net 48 "Net-(R3-Pad2)")
+	(net 49 "Net-(R4-Pad2)")
 	(footprint "Connector_USB:USB_C_Receptacle_Amphenol_124019772112A"
 		(layer "F.Cu")
@@
 			(layers "F.Cu" "F.Mask" "F.Paste")
 			(roundrect_rratio 0.25)
-			(net 46 "Net-(SW7-C)")
+			(net 48 "Net-(R3-Pad2)")
 			(pintype "passive")
 		)
@@
 			(layers "F.Cu" "F.Mask" "F.Paste")
 			(roundrect_rratio 0.25)
-			(net 9 "Net-(SW4-C)")
+			(net 49 "Net-(R4-Pad2)")
 			(pintype "passive")
 		)

Commit message: pcb changes
Parts:
- SW4, SW7: footprint Button_Switch_SMD:Nidec_Copal_CAS-120A -> Switch:SW_500SDP1S1M2QEA
- moved C1 17.0 mm to (106.8, 126.6)
- moved C2 17.0 mm to (101.6, 132.2)
- moved C21 17.0 mm to (113.8, 153.8)
- moved C8 17.0 mm to (102.3, 141.0)
- moved C9 17.0 mm to (104.8, 154.0)
- moved D5 17.0 mm to (101.2, 127.6)
- moved J9 17.0 mm to (110.0, 136.6)
- moved R13 17.0 mm to (101.0, 124.0)
- moved R18 17.0 mm to (103.8, 145.6)
- moved R19 17.0 mm to (118.8, 150.0)
- moved R20 17.0 mm to (109.0, 154.2)
- moved R21 17.0 mm to (115.8, 150.0)
- moved R22 17.0 mm to (111.6, 130.8)
- moved R23 17.0 mm to (111.6, 127.5)
- moved R3 17.0 mm to (112.4, 150.4)
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Routing:
- net V3.3: track 157.8 -> 136.8 mm
- net Net-(J3-In): track 36.1 -> 15.7 mm
- net Net-(SW4-A): track 3.86 -> 15.0 mm
- net Net-(J7-In): track 35.9 -> 27.7 mm
Other:
- board text added: "DESIGNED BY:"
- board text added: "Ethan Marreel Jordan Savin Daniel Stucker"
- board text removed: "DESIGNED BY: Ethan Marreel Jordan Savin Daniel Stucker"
