File: Osciliscope.kicad_sch (KiCad schematic)
At the start: 62 parts, among them J1 Conn_01x03_Socket, J10 Conn_01x01_Socket, J2 Conn_01x04_Socket, J3 U.FL, J4 Conn_01x04_Socket, J5 USB_C_Receptacle_USB2.0_14P, J6 Conn_01x02_MountingPin, J7 U.FL, J8 Conn_01x03_Socket, J9 Conn_01x03_Socket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

Commit message: Changes
Parts:
- removed J1, J8, J9: Conn_01x03_Socket, symbol Connector:Conn_01x03_Socket
- removed J10: Conn_01x01_Socket, symbol Connector:Conn_01x01_Socket
- added J1: Conn_01x09_Socket, symbol Connector:Conn_01x09_Socket
Connections:
- net Ch1_vis: now also J1.9 (Pin_9)
- net Ch2_vis: now also J1.8 (Pin_8)
- net H_clk: now also J1.7 (Pin_7)
- net H_dt: now also J1.6 (Pin_6)
- net Trig_ch: now also J1.3 (Pin_3)
- net Trig_clk: now also J1.2 (Pin_2)
- net Trig_dt: now also J1.1 (Pin_1)
- net V_clk: now also J1.5 (Pin_5)
- net V_dt: now also J1.4 (Pin_4)
- net at R3.2: no longer SW3.2 (B)

Commit message: front end improvements
Parts:
- added C20: 20pF, Capacitor_SMD:C_1206_3216Metric, symbol Device:C
- added R10: 5k, Capacitor_SMD:C_0603_1608Metric, symbol Device:R
- added R21: 1M, Capacitor_SMD:C_0603_1608Metric, symbol Device:R
- R14, R20: value 100k -> 1M
- R18: value 1M -> 5k
Connections:
- net C1_G_IN: now also R18.2
- net C1_G_OUT: now also R18.1
- net C2_G_IN: now also R10.2
- net C2_G_OUT: now also R10.1
- net GND: now also R14.1, R20.1, C20.1; no longer R14.2, R20.2
- net at C9.1, R19.1, SW3.3 (A): now also J7.1 (In), R20.2; no longer R20.1
- net at R19.2: now also C9.2, SW3.1 (C); no longer J7.1 (In)
- net at C10.2, SW4.1 (C): now also R21.2
- net at C10.1, SW4.3 (A): now also J3.1 (In), R14.2, C20.2, R21.1; no longer R14.1, R18.1
- net at R3.2: now also SW3.2 (B)
Other:
- moved on the sheet: C10, C9, J3, SW3, SW4

Commit message: updates to schematic
Parts:
- added C21: 20pF, Capacitor_SMD:C_1206_3216Metric, symbol Device:C
- added TP1: TestPoint, symbol Connector:TestPoint
- added U6: TLV9061xDBV, Package_TO_SOT_SMD:SOT-23-5, symbol Amplifier_Operational:TLV9061xDBV
Connections:
- net GND: now also R19.2, R21.2, C21.1, U6.2 (V-)
- net V3.3: now also U6.5 (V+)
- net at C9.1, J7.1 (In), R20.2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: now also C21.2, TP1.1; no longer R19.1
- net at C10.1, C20.2, J3.1 (In)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: no longer R21.1
- net at C10.2, SW4.1 (C): now also R21.1; no longer R21.2
- net at C9.2, SW3.1 (C): now also R19.1; no longer R19.2
- net V1.8: no longer names the net of C4.2, C5.1, R11.1, R12.2
- net V1.8: now also U6.3 (+); no longer U5.3 (+), U7.3 (+)
- new net V1.65: U5.3 (+), U6.1, U6.4 (-), U7.3 (+)
Other:
- moved on the sheet: R19, R20

Commit message: more changes to circuit diagram
Parts:
- removed R19, R21: 1M, Capacitor_SMD:C_0603_1608Metric, symbol Device:R
- added SW7, SW8: SW_Nidec_CAS-120A1, Button_Switch_SMD:Nidec_Copal_CAS-120A, symbol Switch:SW_Nidec_CAS-120A1
Connections:
- net at C21.2, J7.1 (In), R20.2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: now also SW7.2 (B); no longer C9.1, SW3.3 (A)
- net at C10.2: now also SW8.1 (C); no longer SW4.1 (C)
- net at R4.2: now also SW8.2 (B); no longer SW4.2 (B)
- net at C20.2, J3.1 (In), R14.2: now also SW4.2 (B); no longer C10.1, SW4.3 (A)
- new net: SW4.1 (C), SW8.3 (A)
- new net: SW3.3 (A), SW7.1 (C)
- new net: C9.1, SW7.3 (A)
- new net: C10.1, SW4.3 (A)
Other:
- note added: "additional attenuation?????"
- moved on the sheet: C11, C12, C13, C3, C4, C5, C9, D5, J2, J5, J6, R11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

Commit message: DOUBLE POWAH
Parts:
- removed C11: 1uF, Capacitor_SMD:C_1206_3216Metric, symbol Device:C
- removed C12, C13: 10u, Capacitor_SMD:C_1206_3216Metric, symbol Device:C
- removed SW3, SW8: SW_Nidec_CAS-120A1, Button_Switch_SMD:Nidec_Copal_CAS-120A, symbol Switch:SW_Nidec_CAS-120A1
- removed U3: IP2721, Package_SO:TSSOP-16_4.4x5mm_P0.65mm, symbol Interface_USB:IP2721
- removed U4: AZ1084-5.0, Package_TO_SOT_SMD:TO-252-2, symbol Regulator_Linear:AZ1084-5.0
- removed U8: MCP4251-104E/ML-ND, Package_SO:TSSOP-14-1EP_4.4x5mm_P0.65mm, symbol Potentiometer_Digital:MCP4251-xxxx-SL
- added J8: USB_C_Receptacle_USB2.0_14P, Connector_USB:USB_C_Receptacle_Amphenol_124019772112A, symbol Connector:USB_C_Receptacle_USB2.0_14P
- added J9: Conn_01x03_Socket, Connector_PinSocket_2.00mm:PinSocket_1x03_P2.00mm_Vertical, symbol Connector:Conn_01x03_Socket
- added R19, R21, R22, R23: 5.5k, Capacitor_SMD:C_0603_1608Metric, symbol Device:R
- added TP2, TP3, TP4, TP5, TP6: TestPoint, TestPoint:TestPoint_Pad_3.0x3.0mm, symbol Connector:TestPoint
- added U3: CH340N, Package_SO:JEITA_SOIC-8_3.9x4.9mm_P1.27mm, symbol Interface_USB:CH340N
- J1: footprint (none) -> Connector_PinSocket_2.00mm:PinSocket_1x09_P2.00mm_Vertical
- J6: footprint (none) -> Connector_PinSocket_2.00mm:PinSocket_1x02_P2.00mm_Vertical
- TP1: footprint (none) -> TestPoint:TestPoint_Pad_3.0x3.0mm
Connections:
- net USBCRAW is gone; now on net 5Vin: J5.A4 (VBUS), J5.A9 (VBUS), J5.B4 (VBUS), J5.B9 (VBUS)
- net 5Vin: now also J8.A4 (VBUS), J8.A9 (VBUS), J8.B4 (VBUS), J8.B9 (VBUS), U3.5 (VCC)
- net GND: now also J8.A1 (GND), J8.A12 (GND), J8.B1 (GND), J8.B12 (GND), J8.S1 (SHIELD), R19.1, R21.1, R22.1, R23.1, U3.3 (GND)
- net V1.65: now also TP6.1
- net V3.3: now also TP5.1
- net at J5.A5 (CC1): now also R22.2
- net at J5.B5 (CC2): now also R23.2
- net at C10.2: now also R4.2, SW4.1 (C)
- net V1.65RAW: now reaches C4.2, C5.1, R11.1, R12.2, U6.3 (+)
- net at SW7.1 (C): now also C9.2, R3.2
- net at C20.2, J3.1 (In), R14.2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: now also TP2.1
- net C1_G_IN: no longer names the net of R18.2, R3.1, U5.4 (-)
- net C1_G_OUT renamed CHAN_1
- net CHAN_1: now also TP4.1
- net C2_G_IN: no longer names the net of R10.2, R4.1, U7.4 (-)
- net C2_G_OUT renamed CHAN_2
- net CHAN_2: now also TP3.1
- new net: J8.A5 (CC1), R19.2
- new net: J8.A6 (D+), J8.B6 (D+), U3.1 (UD+)
- new net: J8.A7 (D-), J8.B7 (D-), U3.2 (UD-)
- new net: J8.B5 (CC2), R21.2
- new net RTS: J9.1 (Pin_1), U3.4 (~{RTS})
- new net RXD: J9.2 (Pin_2), U3.7 (RXD)
- new net TXD: J9.3 (Pin_3), U3.6 (TXD)
Other:
- moved on the sheet: J5

Commit message: changes to lots of stuff
Parts:
- removed SW4, SW7: SW_Nidec_CAS-120A1, Button_Switch_SMD:Nidec_Copal_CAS-120A, symbol Switch:SW_Nidec_CAS-120A1
- added S1, S2: 500SDP1S1M2QEA, 500SDP1S1M2QEA:SW_500SDP1S1M2QEA, symbol 500SDP1S1M2QEA:500SDP1S1M2QEA
- C10, C9: footprint Capacitor_SMD:C_1206_3216Metric -> (none)
Connections:
- net at C21.2, J7.1 (In), R20.2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: now also S2.2
- net at C20.2, J3.1 (In), R14.2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: now also S1.2
- net at R3.2: now also S2.5; no longer C9.2
- net at C9.1: now also S2.3
- net at C10.1: now also S1.3
- net at R4.2: now also S1.5; no longer C10.2
- new net: S2.1, S2.4
- new net: C9.2, S2.6
- new net: S1.1, S1.4
- new net: C10.2, S1.6
Other:
- note removed: "additional attenuation?????"
- moved on the sheet: C20, J3, R10, R14, R18, R3, R4, TP2, TP3, TP4, U5, U7

Commit message: Footprint updates
Parts:
- C1, C14, C15, C16, C17, C18, C19, C2, C20, C21, C3, C4, C5, C6, C7, C8: footprint Capacitor_SMD:C_1206_3216Metric -> Capacitor_SMD:C_0402_1005Metric
- C10, C9: footprint (none) -> Capacitor_SMD:C_0402_1005Metric
- D5: footprint PCM_JLCPCB:D_0805 -> Capacitor_SMD:C_0603_1608Metric
- R13: value 10k -> 1k
Changed lines of the file:
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@@
 			)
 		)
-		(property "Footprint" "Capacitor_SMD:C_1206_3216Metric"
+		(property "Footprint" "Capacitor_SMD:C_0402_1005Metric"
 			(at 72.0852 33.02 0)
 			(effects
@@
 			)
 		)
-		(property "Footprint" "Capacitor_SMD:C_1206_3216Metric"
+		(property "Footprint" "Capacitor_SMD:C_0402_1005Metric"
 			(at 272.7452 63.5 0)
 			(effects
@@
 			)
 		)
-		(property "Footprint" "Capacitor_SMD:C_1206_3216Metric"
+		(property "Footprint" "Capacitor_SMD:C_0402_1005Metric"
 			(at 36.5252 55.88 0)
 			(effects
@@
 			)
 		)
-		(property "Footprint" "Capacitor_SMD:C_1206_3216Metric"
+		(property "Footprint" "Capacitor_SMD:C_0402_1005Metric"
 			(at 249.8852 123.19 0)
 			(effects
@@
 			)
 		)
-		(property "Footprint" "Capacitor_SMD:C_1206_3216Metric"
+		(property "Footprint" "Capacitor_SMD:C_0402_1005Metric"
 			(at 180.0352 97.79 0)
 			(effects
@@
 			)
 		)
-		(property "Footprint" "PCM_JLCPCB:D_0805"
+		(property "Footprint" "Capacitor_SMD:C_0603_1608Metric"
 			(at 144.78 145.288 90)
 			(effects
@@
 			)
 		)
-		(property "Footprint" "Capacitor_SMD:C_1206_3216Metric"
+		(property "Footprint" "Capacitor_SMD:C_0402_1005Metric"
 			(at 227.0252 63.5 0)
 			(effects
@@
 			)
 		)
-		(property "Footprint" "Capacitor_SMD:C_1206_3216Metric"
+		(property "Footprint" "Capacitor_SMD:C_0402_1005Metric"
 			(at 42.8752 33.02 0)
 			(effects
@@
 			)
 		)
-		(property "Footprint" "Capacitor_SMD:C_1206_3216Metric"
+		(property "Footprint" "Capacitor_SMD:C_0402_1005Metric"
 			(at 249.8852 63.5 0)
 			(effects
@@
 			)
 		)
-		(property "Footprint" "Capacitor_SMD:C_1206_3216Metric"
+		(property "Footprint" "Capacitor_SMD:C_0402_1005Metric"
 			(at 158.4452 66.04 0)
 			(effects
@@
 			)
 		)
-		(property "Footprint" "Capacitor_SMD:C_1206_3216Metric"
+		(property "Footprint" "Capacitor_SMD:C_0402_1005Metric"
 			(at 158.4452 73.66 0)
 			(effects
@@
 			)
 		)
-		(property "Footprint" "Capacitor_SMD:C_1206_3216Metric"
+		(property "Footprint" "Capacitor_SMD:C_0402_1005Metric"
 			(at 105.1052 33.02 0)
 			(effects
@@
 			)
 		)
-		(property "Footprint" "Capacitor_SMD:C_1206_3216Metric"
+		(property "Footprint" "Capacitor_SMD:C_0402_1005Metric"
 			(at 39.0652 102.87 0)
 			(effects
@@
 			)
 		)
-		(property "Value" "10k"
+		(property "Value" "1k"
 			(at 156.972 140.462 90)
 			(effects
@@
 			)
 		)
-		(property "Footprint" "Capacitor_SMD:C_1206_3216Metric"
+		(property "Footprint" "Capacitor_SMD:C_0402_1005Metric"
 			(at 204.1652 63.5 0)
 			(effects
@@
 		(on_board yes)
 		(dnp no)
-		(fields_autoplaced yes)
 		(property "Reference" "J4"
 			(at 45.72 156.2099 0)
@@
 			)
 		)
-		(property "Footprint" "Capacitor_SMD:C_1206_3216Metric"
+		(property "Footprint" "Capacitor_SMD:C_0402_1005Metric"
 			(at 272.7452 123.19 0)
 			(effects
@@
 			)
 		)
-		(property "Footprint" "Capacitor_SMD:C_1206_3216Metric"
+		(property "Footprint" "Capacitor_SMD:C_0402_1005Metric"
 			(at 94.9452 33.02 0)
 			(effects
@@
 			)
 		)
-		(property "Footprint" "Capacitor_SMD:C_1206_3216Metric"
+		(property "Footprint" "Capacitor_SMD:C_0402_1005Metric"
 			(at 83.5152 33.02 0)
 			(effects
@@
 		(on_board yes)
 		(dnp no)
-		(fields_autoplaced yes)
 		(property "Reference" "R18"
-			(at 99.06 64.77 90)
+			(at 99.314 75.184 90)
 			(effects
 				(font
@@
 		)
 		(property "Value" "5k"
-			(at 99.06 67.31 90)
+			(at 99.314 77.724 90)
 			(effects
 				(font
@@
 			)
 		)
-		(property "Footprint" ""
+		(property "Footprint" "Capacitor_SMD:C_0402_1005Metric"
 			(at 60.96 77.7748 0)
 			(effects
@@
 			)
 		)
-		(property "Footprint" ""
+		(property "Footprint" "Capacitor_SMD:C_0402_1005Metric"
 			(at 67.31 126.0348 0)
 			(effects

Commit message: pcb changes
Parts:
- added TP7, TP8: TestPoint, TestPoint:TestPoint_Pad_3.0x3.0mm, symbol Connector:TestPoint
Connections:
- net at R10.2, R4.1, U7.4 (-): now also TP8.1
- net at R18.2, R3.1, U5.4 (-): now also TP7.1
Changed lines of the file:
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@@
 	)
 	(junction
+		(at 86.36 60.96)
+		(diameter 0)
+		(color 0 0 0 0)
+	)
+	(junction
 		(at 96.52 20.32)
 		(diameter 0)
@@
 	)
 	(junction
+		(at 95.25 119.38)
+		(diameter 0)
+		(color 0 0 0 0)
+	)
+	(junction
 		(at 154.94 152.4)
 		(diameter 0)
@@
 	(wire
 		(pts
+			(xy 93.98 119.38) (xy 95.25 119.38)
+		)
+		(stroke
+			(width 0)
+			(type default)
+		)
+	)
+	(wire
+		(pts
 			(xy 88.9 55.88) (xy 93.98 55.88)
 		)
@@
 	(wire
 		(pts
-			(xy 82.55 60.96) (xy 88.9 60.96)
+			(xy 82.55 60.96) (xy 86.36 60.96)
 		)
 		(stroke
@@
 	(wire
 		(pts
+			(xy 86.36 60.96) (xy 88.9 60.96)
+		)
+		(stroke
+			(width 0)
+			(type default)
+		)
+	)
+	(wire
+		(pts
 			(xy 95.25 121.92) (xy 102.87 121.92)
 		)
@@
 	(wire
 		(pts
-			(xy 95.25 109.22) (xy 95.25 121.92)
+			(xy 95.25 109.22) (xy 95.25 119.38)
 		)
 		(stroke
@@
 	(wire
 		(pts
+			(xy 95.25 119.38) (xy 95.25 121.92)
+		)
+		(stroke
+			(width 0)
+			(type default)
+		)
+	)
+	(wire
+		(pts
 			(xy 129.54 160.02) (xy 128.27 160.02)
 		)
@@
 	)
 	(symbol
+		(lib_id "Connector:TestPoint")
+		(at 86.36 60.96 180)
+		(unit 1)
+		(exclude_from_sim no)
+		(in_bom yes)
+		(on_board yes)
+		(dnp no)
+		(fields_autoplaced yes)
+		(property "Reference" "TP7"
+			(at 88.9 62.9919 0)
+			(effects
+				(font
+					(size 1.27 1.27)
+				)
+				(justify right)
+			)
+		)
+		(property "Value" "TestPoint"
+			(at 88.9 65.5319 0)
+			(effects
+				(font
+					(size 1.27 1.27)
+				)
+				(justify right)
+			)
+		)
+		(property "Footprint" "TestPoint:TestPoint_Pad_3.0x3.0mm"
+			(at 81.28 60.96 0)
+			(effects
+				(font
+					(size 1.27 1.27)
+				)
+				(hide yes)
+			)
+		)
+		(property "Datasheet" "~"
+			(at 81.28 60.96 0)
+			(effects
+				(font
+					(size 1.27 1.27)
+				)
+				(hide yes)
+			)
+		)
+		(property "Description" "test point"
+			(at 86.36 60.96 0)
+			(effects
+				(font
+					(size 1.27 1.27)
+				)
+				(hide yes)
+			)
+		)
+		(pin "1"
+		)
+		(instances
+			(project "Osciliscope"
+				(path "/8c683ef5-a777-4de0-90bd-818351a6a189"
+					(reference "TP7")
+					(unit 1)
+				)
+			)
+		)
+	)
+	(symbol
 		(lib_id "power:GND")
 		(at 71.12 191.77 0)
@@
 					(unit 1)
 				)
+			)
+		)
+	)
+	(symbol
+		(lib_id "Connector:TestPoint")
+		(at 93.98 119.38 90)
+		(unit 1)
+		(exclude_from_sim no)
+		(in_bom yes)
+		(on_board yes)
+		(dnp no)
+		(fields_autoplaced yes)
+		(property "Reference" "TP8"
+			(at 90.678 114.3 90)
+			(effects
+				(font
+					(size 1.27 1.27)
+				)
+			)
+		)
+		(property "Value" "TestPoint"
+			(at 90.678 116.84 90)
+			(effects
+				(font
+					(size 1.27 1.27)
+				)
+			)
+		)
+		(property "Footprint" "TestPoint:TestPoint_Pad_3.0x3.0mm"
+			(at 93.98 114.3 0)
+			(effects
+				(font
+					(size 1.27 1.27)
+				)
+				(hide yes)
+			)
+		)
+		(property "Datasheet" "~"
+			(at 93.98 114.3 0)
+			(effects
+				(font
+					(size 1.27 1.27)
+				)
+				(hide yes)
+			)
+		)
+		(property "Description" "test point"
+			(at 93.98 119.38 0)
+			(effects
+				(font
+					(size 1.27 1.27)
+				)
+				(hide yes)
+			)
+		)
+		(pin "1"
+		)
+		(instances
+			(project "Osciliscope"
+				(path "/8c683ef5-a777-4de0-90bd-818351a6a189"
+					(reference "TP8")
+					(unit 1)
+				)
